File: Hardware/Panel/gearseq_panel/gearseq_panel.kicad_pcb (KiCad board)
At the start: 2 copper layers, 100 x 200 mm, 28 parts

Commit message: Panel design
Parts:
- removed H14: Led_Hole, Kosmo_panel:Kosmo_LED_Hole
- removed H16, H17: Pot_Hole, Kosmo_panel:Kosmo_Pot_Hole
- GRAF1: footprint gapseq:gapseq_panel_holes -> gearseq_panel:gearseq_panel_holes
- GRAF2: footprint gapseq:gapseq_panel_art -> gearseq_panel:gearseq_panel_art
- GRAF3: value Graphic -> CC0 logo
- H12: value Led_Hole -> Push_Button_Hole; footprint Kosmo_panel:Kosmo_LED_Hole -> Kosmo_panel:Push_Button_A-3487
- H13: value Led_Hole -> Jack_Hole; footprint Kosmo_panel:Kosmo_LED_Hole -> Kosmo_panel:Kosmo_Jack_Hole
- H4: value Pot_Hole -> Push_Button_Hole; footprint Kosmo_panel:Kosmo_Pot_Hole -> Kosmo_panel:Push_Button_A-3487
- moved H22 120.0 mm to (12.5, 30.0)
- moved H21 93.4 mm to (12.5, 60.0)
- moved H13 90.9 mm to (12.5, 90.0)
- moved H19 79.1 mm to (12.5, 175.0)
- moved H12 62.7 mm to (12.5, 150.0)
- moved H4 61.3 mm to (37.5, 150.0)
- moved H18 58.3 mm to (12.5, 120.0)
- moved OLED1 57.0 mm to (75.0, 60.0)
- moved H9 55.9 mm to (25.0, 180.0)
- moved H5 52.0 mm to (37.5, 60.0)
- moved H2 42.5 mm to (37.5, 120.0)
- moved H6 32.5 mm to (37.5, 90.0)
- moved H15 30.4 mm to (75.0, 90.0)
- moved H7 15.0 mm to (25.0, 170.0)
- moved H3 12.5 mm to (37.5, 30.0)
Connections:
- H12 pad 1: (no net) -> GND
- H13 pad 1: (no net) -> GND
Other:
- outline, holes or cut-outs redrawn
- board text added: "Algorithm pot"
- board text added: "CV1 jack"
- board text added: "CV1 pot"
- board text added: "CV2 jack"
- board text added: "CV2 pot"
- board text added: "CV3 jack"
- board text added: "CV3 pot"
- board text added: "CV4 jack"
- board text added: "CV4 pot"
- board text added: "OLED"
- board text added: "Panel design by Rich Holmes October 2021 CC0 1.0 JLCJLCJLCJLC"
- board text added: "Period LED"
- board text added: "Period jack"
- board text added: "Reset LED"
- board text added: "Reset jack"
- board text added: "Reset push button"
- board text added: "Sequence LED"
- board text added: "Sequence jack"
- board text added: "Step LED"
- board text added: "Step jack"
- board text added: "Step push button"
- board text removed: "Panel design by Rich Holmes August 2021 CC0 1.0 JLCJLCJLCJLC"
