File: Hardware/Panel/gearseq_panel/gearseq_panel.kicad_pcb (KiCad board)
At the start: 2 copper layers, 100 x 200 mm, 25 parts

Commit message: Final pre fab tweaks, correct oversize LED footprint
Parts:
- added H14: Switch_Hole, Kosmo_panel:Kosmo_Switch_Hole, F.Cu at (75.0, 120.0)
- turned OLED1 to 180 degrees
Other:
- board text added: "Display switch"
